Commit message: Update URDF

File: lobot_description/urdf/xarm.gazebo.xacro (robot description, xacro)
@@ -20,3 +20,9 @@
     </inertial>
   </xacro:macro>
+  <!-- ros_control plugin -->
+  <gazebo>
+    <plugin name="gazebo_ros_control" filename="libgazebo_ros_control.so">
+      <robotNamespace>/arm</robotNamespace>
+    </plugin>
+  </gazebo>
 </robot>

File: lobot_description/urdf/xarm.urdf.xacro (robot description, xacro)
@@ -238,4 +238,5 @@
     <axis xyz="0 1 0" />
     <limit lower="-0.025" upper="0" effort="16" velocity="2" />
+    <mimic joint="gripper_joint1" multiplier="-1" />
   </joint>
 </robot>

Commit message: Update URDF

File: lobot_description/urdf/xarm.gazebo.xacro (robot description, xacro)
@@ -6,16 +6,16 @@
       <mass value="${mass}" />
       <inertia
-        ixx="${0.01 * mass * length * width * height}" ixy="0" ixz="0"
-        iyy="${0.01 * mass * length * width * height}" iyz="0"
-        izz="${0.1 * mass * length * width * height}" />
+        ixx="1" ixy="0" ixz="0"
+        iyy="0.5" iyz="0"
+        izz="1" />
     </inertial>
   </xacro:macro>
   <xacro:macro name="cylinder_inertial_matrix" params="radius length mass *origin">
     <inertial>
-      <mass value="{mass}" />
+      <mass value="${mass}" />
       <inertia
-        ixx="${0.05 * mass * (3 * radius * radius + length * length)}" ixy="0" ixz="0"
-        iyy="${0.05 * mass * (3 * radius * radius + length * length)}" iyz="0"
-        izz="${0.5 * mass * radius * radius}" />
+        ixx="1" ixy="0" ixz="0"
+        iyy="0.5" iyz="0"
+        izz="1" />
     </inertial>
   </xacro:macro>
@@ -23,6 +23,33 @@
   <gazebo>
     <plugin name="gazebo_ros_control" filename="libgazebo_ros_control.so">
-      <robotNamespace>/arm</robotNamespace>
+      <robotNamespace>/xarm</robotNamespace>
     </plugin>
   </gazebo>
+  <gazebo reference="base_link">
+    <material>Gazebo/Black</material>
+  </gazebo>
+  <gazebo reference="arm_link1">
+    <material>Gazebo/Orange</material>
+  </gazebo>
+  <gazebo reference="arm_link2">
+    <material>Gazebo/Orange</material>
+  </gazebo>
+  <gazebo reference="arm_link3">
+    <material>Gazebo/Orange</material>
+  </gazebo>
+  <gazebo reference="arm_link4">
+    <material>Gazebo/Orange</material>
+  </gazebo>
+  <gazebo reference="arm_link5">
+    <material>Gazebo/Orange</material>
+  </gazebo>
+  <gazebo reference="gripper_link">
+    <material>Gazebo/Red</material>
+  </gazebo>
+  <gazebo reference="left_gripper">
+    <material>Gazebo/Red</material>
+  </gazebo>
+  <gazebo reference="right_gripper">
+    <material>Gazebo/Red</material>
+  </gazebo>
 </robot>

File: lobot_description/urdf/xarm.urdf.xacro (robot description, xacro)
@@ -24,9 +24,9 @@
   </xacro:property>
   <!-- arm_link1 properties -->
+  <xacro:property name="arm_link1_radius" value="0.045" />
   <xacro:property name="arm_link1_length" value="0.05" />
-  <xacro:property name="arm_link1_radius" value="0.045" />
   <xacro:property name="arm_link1_geometry_origin">
     <geometry>
-      <cylinder length="${arm_link1_length}" radius="${arm_link1_radius}" />
+      <cylinder radius="${arm_link1_radius}" length="${arm_link1_length}" />
     </geometry>
     <origin xyz="0 0 ${arm_link1_length/2}" rpy="0 0 0" />
@@ -63,9 +63,9 @@
   </xacro:property>
   <!-- arm_link5 properties -->
+  <xacro:property name="arm_link5_radius" value="0.016" />
   <xacro:property name="arm_link5_length" value="0.05" />
-  <xacro:property name="arm_link5_radius" value="0.016" />
   <xacro:property name="arm_link5_geometry_origin">
     <geometry>
-      <cylinder length="${arm_link5_length}" radius="${arm_link5_radius}" />
+      <cylinder radius="${arm_link5_radius}" length="${arm_link5_length}" />
     </geometry>
     <origin xyz="0 0 ${arm_link5_length/2}" rpy="0 0 0" />
@@ -91,4 +91,11 @@
     <origin xyz="0 0 ${gripper_height/2}" rpy="0 0 0" />
   </xacro:property>
+  <!-- Used to fix robot to Gazebo -->
+  <link name="dummy_base" />
+  <joint name="fixed" type="fixed">
+    <origin xyz="0 0 0" rpy="0 0 0" />
+    <parent link="dummy_base" />
+    <child link="base_link" />
+  </joint>
   <!--////////// BASE_LINK //////////-->
   <link name="base_link">
@@ -113,4 +120,7 @@
       <xacro:insert_block name="arm_link1_geometry_origin" />
     </collision>
+    <xacro:cylinder_inertial_matrix radius="${arm_link1_radius}" length="${arm_link1_length}" mass="${base_mass}">
+      <origin xyz="0 0 0" rpy="0 0 0" />
+    </xacro:cylinder_inertial_matrix>
   </link>
   <joint name="arm_joint1" type="revolute">
@@ -120,5 +130,5 @@
     <axis xyz="0 0 1" />
     <limit lower="${-pi*2/3}" upper="${pi*2/3}" effort="16" velocity="2.5" />
-    <dynamics damping="0" friction="0"/>
+    <dynamics damping="50" friction="1"/>
   </joint>
   <!--////////// ARM_LINK2 //////////-->
@@ -131,4 +141,7 @@
       <xacro:insert_block name="arm_link2_geometry_origin" />
     </collision>
+    <xacro:box_inertial_matrix length="${arm_link2_length}" width="${arm_link2_width}" height="${arm_link2_height}" mass="${base_mass}">
+      <origin xyz="0 0 0" rpy="0 0 0" />
+    </xacro:box_inertial_matrix>
   </link>
   <joint name="arm_joint2" type="revolute">
@@ -148,4 +161,7 @@
       <xacro:insert_block name="arm_link3_geometry_origin" />
     </collision>
+    <xacro:box_inertial_matrix length="${arm_link3_length}" width="${arm_link3_width}" height="${arm_link3_height}" mass="${base_mass}">
+      <origin xyz="0 0 0" rpy="0 0 0" />
+    </xacro:box_inertial_matrix>
   </link>
   <joint name="arm_joint3" type="revolute">
@@ -165,4 +181,7 @@
       <xacro:insert_block name="arm_link4_geometry_origin" />
     </collision>
+    <xacro:box_inertial_matrix length="${arm_link4_length}" width="${arm_link4_width}" height="${arm_link4_height}" mass="${base_mass}">
+      <origin xyz="0 0 0" rpy="0 0 0" />
+    </xacro:box_inertial_matrix>
   </link>
   <joint name="arm_joint4" type="revolute">
@@ -182,4 +201,7 @@
       <xacro:insert_block name="arm_link5_geometry_origin" />
     </collision>
+    <xacro:cylinder_inertial_matrix radius="${arm_link5_radius}" length="${arm_link5_length}" mass="${base_mass}">
+      <origin xyz="0 0 0" rpy="0 0 0" />
+    </xacro:cylinder_inertial_matrix>
   </link>
   <joint name="arm_joint5" type="revolute">
@@ -199,4 +221,7 @@
       <xacro:insert_block name="gripper_link_geometry_origin" />
     </collision>
+    <xacro:box_inertial_matrix length="${gripper_link_length}" width="${gripper_link_width}" height="${gripper_link_height}" mass="${base_mass}">
+      <origin xyz="0 0 0" rpy="0 0 0" />
+    </xacro:box_inertial_matrix>
   </link>
   <joint name="arm_to_gripper" type="fixed">
@@ -214,4 +239,7 @@
       <xacro:insert_block name="gripper_geometry_origin" />
     </collision>
+    <xacro:box_inertial_matrix length="${gripper_length}" width="${gripper_width}" height="${gripper_height}" mass="${base_mass}">
+      <origin xyz="0 0 0" rpy="0 0 0" />
+    </xacro:box_inertial_matrix>
   </link>
   <joint name="gripper_joint1" type="prismatic">
@@ -223,5 +251,5 @@
   </joint>
   <!--////////// RIGHT_GRIPPER //////////-->
-  <link name="right_rigpper">
+  <link name="right_gripper">
     <visual>
       <xacro:insert_block name="gripper_geometry_origin" />
@@ -231,9 +259,12 @@
       <xacro:insert_block name="gripper_geometry_origin" />
     </collision>
+    <xacro:box_inertial_matrix length="${gripper_length}" width="${gripper_width}" height="${gripper_height}" mass="${base_mass}">
+      <origin xyz="0 0 0" rpy="0 0 0" />
+    </xacro:box_inertial_matrix>
   </link>
   <joint name="gripper_joint2" type="prismatic">
     <origin rpy="0 0 0" xyz="0 ${gripper_link_width/2} 0" />
     <parent link="gripper_link" />
-    <child link="right_rigpper" />
+    <child link="right_gripper" />
     <axis xyz="0 1 0" />
     <limit lower="-0.025" upper="0" effort="16" velocity="2" />
