Commit message: Fix errors

File: lobot_description/urdf/xarm.transmission.xacro (robot description, xacro)
@@ -5,9 +5,10 @@
       <type>transmission_interface/SimpleTransmission</type>
       <joint name="${joint_name}">
+        <!-- hardwareInterface must be EffortJointInterface when this transmission is loaded in Gazebo -->
+        <!-- <hardwareInterface>hardware_interface/EffortJointInterface</hardwareInterface> -->
         <hardwareInterface>hardware_interface/PositionJointInterface</hardwareInterface>
       </joint>
       <actuator name="motor">
         <mechanicalReduction>1</mechanicalReduction>
-        <hardwareInterface>hardware_interface/PositionJointInterface</hardwareInterface>
       </actuator>
     </transmission>

File: lobot_description/urdf/xarm.urdf.xacro (robot description, xacro)
@@ -107,5 +107,5 @@
       <xacro:insert_block name="base_link_geometry_origin" />
     </collision>
-    <xacro:box_inertial_matrix length="${base_link_length}" width="${base_link_width}" height="${base_link_height}" mass="${base_mass}">
+    <xacro:box_inertial_matrix length="${base_link_length}" width="${base_link_width}" height="${base_link_height}" mass="2*${base_mass}">
       <origin xyz="0 0 0" rpy="0 0 0" />
     </xacro:box_inertial_matrix>
@@ -120,5 +120,5 @@
       <xacro:insert_block name="arm_link1_geometry_origin" />
     </collision>
-    <xacro:cylinder_inertial_matrix radius="${arm_link1_radius}" length="${arm_link1_length}" mass="${base_mass}">
+    <xacro:cylinder_inertial_matrix radius="${arm_link1_radius}" length="${arm_link1_length}" mass="0.5*${base_mass}">
       <origin xyz="0 0 0" rpy="0 0 0" />
     </xacro:cylinder_inertial_matrix>
@@ -141,5 +141,5 @@
       <xacro:insert_block name="arm_link2_geometry_origin" />
     </collision>
-    <xacro:box_inertial_matrix length="${arm_link2_length}" width="${arm_link2_width}" height="${arm_link2_height}" mass="${base_mass}">
+    <xacro:box_inertial_matrix length="${arm_link2_length}" width="${arm_link2_width}" height="${arm_link2_height}" mass="0.15*${base_mass}">
       <origin xyz="0 0 0" rpy="0 0 0" />
     </xacro:box_inertial_matrix>
@@ -151,4 +151,5 @@
     <axis xyz="0 1 0" />
     <limit lower="${-pi/2}" upper="${pi/2}" effort="16" velocity="2" />
+    <dynamics damping="50" friction="1"/>
   </joint>
   <!--////////// ARM_LINK3 //////////-->
@@ -161,5 +162,5 @@
       <xacro:insert_block name="arm_link3_geometry_origin" />
     </collision>
-    <xacro:box_inertial_matrix length="${arm_link3_length}" width="${arm_link3_width}" height="${arm_link3_height}" mass="${base_mass}">
+    <xacro:box_inertial_matrix length="${arm_link3_length}" width="${arm_link3_width}" height="${arm_link3_height}" mass="0.15*${base_mass}">
       <origin xyz="0 0 0" rpy="0 0 0" />
     </xacro:box_inertial_matrix>
@@ -171,4 +172,5 @@
     <axis xyz="0 1 0" />
     <limit lower="-2" upper="2" effort="16" velocity="2" />
+    <dynamics damping="50" friction="1"/>
   </joint>
   <!--////////// ARM_LINK4 //////////-->
@@ -181,5 +183,5 @@
       <xacro:insert_block name="arm_link4_geometry_origin" />
     </collision>
-    <xacro:box_inertial_matrix length="${arm_link4_length}" width="${arm_link4_width}" height="${arm_link4_height}" mass="${base_mass}">
+    <xacro:box_inertial_matrix length="${arm_link4_length}" width="${arm_link4_width}" height="${arm_link4_height}" mass="0.07*${base_mass}">
       <origin xyz="0 0 0" rpy="0 0 0" />
     </xacro:box_inertial_matrix>
@@ -191,4 +193,5 @@
     <axis xyz="0 1 0" />
     <limit lower="-2" upper="2" effort="16" velocity="2" />
+    <dynamics damping="50" friction="1"/>
   </joint>
   <!--////////// ARM_LINK5 //////////-->
@@ -201,5 +204,5 @@
       <xacro:insert_block name="arm_link5_geometry_origin" />
     </collision>
-    <xacro:cylinder_inertial_matrix radius="${arm_link5_radius}" length="${arm_link5_length}" mass="${base_mass}">
+    <xacro:cylinder_inertial_matrix radius="${arm_link5_radius}" length="${arm_link5_length}" mass="0.07${base_mass}">
       <origin xyz="0 0 0" rpy="0 0 0" />
     </xacro:cylinder_inertial_matrix>
@@ -211,4 +214,5 @@
     <axis xyz="0 0 1" />
     <limit lower="${-pi*2/3}" upper="${pi*2/3}" effort="16" velocity="2.5" />
+    <dynamics damping="50" friction="1"/>
   </joint>
   <!--////////// GRIPPER_LINK //////////-->
@@ -221,5 +225,5 @@
       <xacro:insert_block name="gripper_link_geometry_origin" />
     </collision>
-    <xacro:box_inertial_matrix length="${gripper_link_length}" width="${gripper_link_width}" height="${gripper_link_height}" mass="${base_mass}">
+    <xacro:box_inertial_matrix length="${gripper_link_length}" width="${gripper_link_width}" height="${gripper_link_height}" mass="0.05*${base_mass}">
       <origin xyz="0 0 0" rpy="0 0 0" />
     </xacro:box_inertial_matrix>
@@ -239,5 +243,5 @@
       <xacro:insert_block name="gripper_geometry_origin" />
     </collision>
-    <xacro:box_inertial_matrix length="${gripper_length}" width="${gripper_width}" height="${gripper_height}" mass="${base_mass}">
+    <xacro:box_inertial_matrix length="${gripper_length}" width="${gripper_width}" height="${gripper_height}" mass="0.02*${base_mass}">
       <origin xyz="0 0 0" rpy="0 0 0" />
     </xacro:box_inertial_matrix>
@@ -249,4 +253,5 @@
     <axis xyz="0 1 0" />
     <limit lower="0" upper="0.025" effort="16" velocity="2" />
+    <dynamics damping="50" friction="1"/>
   </joint>
   <!--////////// RIGHT_GRIPPER //////////-->
@@ -259,5 +264,5 @@
       <xacro:insert_block name="gripper_geometry_origin" />
     </collision>
-    <xacro:box_inertial_matrix length="${gripper_length}" width="${gripper_width}" height="${gripper_height}" mass="${base_mass}">
+    <xacro:box_inertial_matrix length="${gripper_length}" width="${gripper_width}" height="${gripper_height}" mass="0.02*${base_mass}">
       <origin xyz="0 0 0" rpy="0 0 0" />
     </xacro:box_inertial_matrix>
@@ -270,4 +275,5 @@
     <limit lower="-0.025" upper="0" effort="16" velocity="2" />
     <mimic joint="gripper_joint1" multiplier="-1" />
+    <dynamics damping="50" friction="1"/>
   </joint>
 </robot>
