Commit message: Add Gazebo properties

File: lobot_description/urdf/xarm.urdf.xacro (robot description, xacro)
@@ -1,5 +1,6 @@
 <?xml version="1.0"?>
-<robot xmlns:xacro="http://www.ros.org/wiki/xacro" name="xarm">
+<robot xmlns:xacro="http://wiki.ros.org/xacro" name="xarm">
   <xacro:include filename="$(find lobot_description)/urdf/xarm.transmission.xacro" />
+  <xacro:include filename="$(find lobot_description)/urdf/xarm.gazebo.xacro" />
   <!-- Define the colors used in this robot -->
   <material name="Black">
@@ -99,4 +100,7 @@
       <xacro:insert_block name="base_link_geometry_origin" />
     </collision>
+    <xacro:box_inertial_matrix length="${base_link_length}" width="${base_link_width}" height="${base_link_height}" mass="${base_mass}">
+      <origin xyz="0 0 0" rpy="0 0 0" />
+    </xacro:box_inertial_matrix>
   </link>
   <!--////////// ARM_LINK1 //////////-->
@@ -116,4 +120,5 @@
     <axis xyz="0 0 1" />
     <limit lower="${-pi*2/3}" upper="${pi*2/3}" effort="16" velocity="2.5" />
+    <dynamics damping="0" friction="0"/>
   </joint>
   <!--////////// ARM_LINK2 //////////-->

Commit message: Update URDF

File: lobot_description/urdf/xarm.urdf.xacro (robot description, xacro)
@@ -60,5 +60,5 @@
       <box size="${arm_link4_length} ${arm_link4_width} ${arm_link4_height}" />
     </geometry>
-    <origin rpy="0 0 0" xyz="0 0 ${arm_link4_height/2}" />
+    <origin xyz="0 0 ${arm_link4_height/2}" rpy="0 0 0" />
   </xacro:property>
   <!-- arm_link5 properties -->
@@ -248,5 +248,5 @@
   </link>
   <joint name="gripper_joint1" type="prismatic">
-    <origin rpy="0 0 0" xyz="0 ${-gripper_link_width/2} 0" />
+    <origin rpy="0 0 0" xyz="0 ${-gripper_link_width/2} ${gripper_link_height}" />
     <parent link="gripper_link" />
     <child link="left_gripper" />
@@ -269,5 +269,5 @@
   </link>
   <joint name="gripper_joint2" type="prismatic">
-    <origin rpy="0 0 0" xyz="0 ${gripper_link_width/2} 0" />
+    <origin rpy="0 0 0" xyz="0 ${gripper_link_width/2} ${gripper_link_height}" />
     <parent link="gripper_link" />
     <child link="right_gripper" />

Commit message: Update package: lobot_hardware_interface

File: lobot_description/urdf/xarm.urdf.xacro (robot description, xacro)
@@ -252,5 +252,5 @@
     <child link="left_gripper" />
     <axis xyz="0 1 0" />
-    <limit lower="0" upper="0.025" effort="16" velocity="2" />
+    <limit lower="0" upper="0.03" effort="16" velocity="2" />
     <dynamics damping="50" friction="1"/>
   </joint>
@@ -273,5 +273,5 @@
     <child link="right_gripper" />
     <axis xyz="0 1 0" />
-    <limit lower="-0.025" upper="0" effort="16" velocity="2" />
+    <limit lower="-0.03" upper="0" effort="16" velocity="2" />
     <mimic joint="gripper_joint1" multiplier="-1" />
     <dynamics damping="50" friction="1"/>
