Commit message: Update package: lobot_description

File: lobot_description/urdf/xarm.urdf (robot description, URDF)
Before this commit: robot xarm, 9 links, 8 joints
Joints:
- joint gripper_joint1: limit lower=0 upper=0.025 effort=16 velocity=2 -> lower=0 upper=0.03 effort=16 velocity=2
- joint gripper_joint2: limit lower=-0.025 upper=0 effort=16 velocity=2 -> lower=-0.03 upper=0 effort=16 velocity=2

Commit message: Update package: lobot_hardware_interface

File: lobot_description/urdf/xarm.urdf (robot description, URDF)
Before this commit: robot xarm, 9 links, 8 joints
Joints:
- joint arm_joint3: limit lower=-2 upper=2 effort=16 velocity=2 -> lower=-2.0944 upper=2.0944 effort=16 velocity=2
- joint arm_joint4: limit lower=-2 upper=2 effort=16 velocity=2 -> lower=-2.0944 upper=2.0944 effort=16 velocity=2

File: lobot_description/urdf/xarm.urdf.xacro (robot description, xacro)
@@ -171,5 +171,5 @@
     <child link="arm_link3" />
     <axis xyz="0 1 0" />
-    <limit lower="-2" upper="2" effort="16" velocity="2" />
+    <limit lower="-2.0944" upper="2.0944" effort="16" velocity="2" />
     <dynamics damping="50" friction="1"/>
   </joint>
@@ -192,5 +192,5 @@
     <child link="arm_link4" />
     <axis xyz="0 1 0" />
-    <limit lower="-2" upper="2" effort="16" velocity="2" />
+    <limit lower="-2.0944" upper="2.0944" effort="16" velocity="2" />
     <dynamics damping="50" friction="1"/>
   </joint>

Commit message: Update package: lobot_kinematics

File: lobot_description/urdf/xarm.urdf (robot description, URDF)
Before this commit: robot xarm, 9 links, 8 joints
Joints:
- joint arm_joint3: limit lower=-2.0944 upper=2.0944 effort=16 velocity=2 -> lower=-2.09439510239 upper=2.09439510239 effort=16 velocity=2
- joint arm_joint4: limit lower=-2.0944 upper=2.0944 effort=16 velocity=2 -> lower=-2.09439510239 upper=2.09439510239 effort=16 velocity=2

File: lobot_description/urdf/xarm.urdf.xacro (robot description, xacro)
@@ -171,5 +171,5 @@
     <child link="arm_link3" />
     <axis xyz="0 1 0" />
-    <limit lower="-2.0944" upper="2.0944" effort="16" velocity="2" />
+    <limit lower="${-pi*2/3}" upper="${pi*2/3}" effort="16" velocity="2" />
     <dynamics damping="50" friction="1"/>
   </joint>
@@ -192,5 +192,5 @@
     <child link="arm_link4" />
     <axis xyz="0 1 0" />
-    <limit lower="-2.0944" upper="2.0944" effort="16" velocity="2" />
+    <limit lower="${-pi*2/3}" upper="${pi*2/3}" effort="16" velocity="2" />
     <dynamics damping="50" friction="1"/>
   </joint>
